Commit message: Reenabling camera and lidar

File: chapter_10_codes/sensor_sim_gazebo/urdf/camera.xacro (robot description, xacro)
@@ -1,7 +1,7 @@
 <?xml version="1.0"?>
-<robot name="sensor" xmlns:xacro="http://www.ros.org/wiki/xacro">
+<robot name="sensor2" xmlns:xacro="http://ros.org/wiki/xacro">
 <!-- camera -->
-  <xacro:include filename="$(find sensor_sim_gazebo)/urdf/sensor.xacro"/>
-  <gazebo reference="sensor">
+  <xacro:include filename="$(find sensor_sim_gazebo)/urdf/sensor2.xacro"/>
+  <gazebo reference="sensor2">
     <sensor type="camera" name="camera1">
       <update_rate>30.0</update_rate>

File: chapter_10_codes/sensor_sim_gazebo/urdf/sensor.xacro (robot description, xacro)
@@ -1,4 +1,4 @@
 <?xml version="1.0"?>
-<robot name="sensor" xmlns:xacro="http://www.ros.org/wiki/xacro">
+<robot name="sensor" xmlns:xacro="http://ros.org/wiki/xacro">
   <xacro:property name="height1" value="0.2" />
   <xacro:property name="width" value="0.2" />
@@ -6,5 +6,5 @@
  <!-- Used for fixing robot to Gazebo 'base_link' -->
   <!-- <link name="${parent}"/> -->
-  <joint name="fixed" type="fixed">
+  <joint name="fixed1" type="fixed">
     <parent link="${parent}"/>
     <child link="sensor"/>
