Commit message: Removing nodes that don't build easily and making some stuff work with our robot

File: chapter_10_codes/sensor_sim_gazebo/urdf/imu.xacro (robot description, xacro)
@@ -1,15 +1,48 @@
 <?xml version="1.0"?>
-<robot name="sensor" xmlns:xacro="http://www.ros.org/wiki/xacro">
-<!-- camera -->
-  <xacro:include filename="$(find sensor_sim_gazebo)/urdf/sensor.xacro"/>
-  <gazebo>
-    <plugin name="imu_plugin" filename="libgazebo_ros_imu.so">
-      <alwaysOn>true</alwaysOn>
-      <bodyName>sensor</bodyName>
-      <topicName>imu</topicName>
-      <serviceName>imu_service</serviceName>
-      <gaussianNoise>0.0</gaussianNoise>
-      <updateRate>20.0</updateRate>
-    </plugin>
-  </gazebo>
+<robot name="sensor" xmlns:xacro="http://ros.org/wiki/xacro">
+  <xacro:macro name="imu" params="name parent *origin" >
+    <xacro:include filename="$(find sensor_sim_gazebo)/urdf/sensor.xacro">
+      <parent>${parent}</parent>
+    </xacro:include>
+    <!-- <link name="${name}">
+      <visual>
+        <origin xyz="0 0 0" rpy="0 0 0" />
+        <geometry>
+          <cylinder radius=".07" length=".06"/>
+        </geometry>
+        <material name="white">
+          <color rgba="1 1 1 1" />
+        </material>
+      </visual>
+      <collision>
+        <origin xyz="0 0 0" rpy="0 0 0" />
+        <geometry>
+          <cylinder radius=".07" length=".06"/>
+        </geometry>
+      </collision>
+      <inertial>
+        <origin xyz="0 0 0" />
+        <mass value="0.1" />
+        <inertia ixx="0.1" ixy="0" ixz="0" iyy="0.1" iyz="0" izz="0.1"/>
+      </inertial>
+    </link>
+    <joint name="${name}" type="fixed">
+      <xacro:insert_block name="origin" />
+      <parent link="${parent}"/>
+      <child link="${name}" />
+    </joint>
+    <gazebo reference="${name}" >
+      <material>Gazebo/White</material>
+    </gazebo> -->
+    <gazebo>
+      <plugin name="sensor" filename="libgazebo_ros_imu.so">
+        <alwaysOn>true</alwaysOn>
+        <bodyName>${parent}</bodyName>
+        <topicName>imu</topicName>
+        <serviceName>imu_service</serviceName>
+        <gaussianNoise>0.1</gaussianNoise>
+        <updateRate>20.0</updateRate>
+      </plugin>
+    </gazebo>
+  </xacro:macro>
 </robot>

File: chapter_10_codes/sensor_sim_gazebo/urdf/sensor.xacro (robot description, xacro)
@@ -3,8 +3,9 @@
   <xacro:property name="height1" value="0.2" />
   <xacro:property name="width" value="0.2" />
+  <xacro:property name="parent" value="base_footprint" />
  <!-- Used for fixing robot to Gazebo 'base_link' -->
-  <link name="world"/>
+  <!-- <link name="${parent}"/> -->
   <joint name="fixed" type="fixed">
-    <parent link="world"/>
+    <parent link="${parent}"/>
     <child link="sensor"/>
   </joint>

Commit message: Fixing the link to the GPS instead of the body. Helps performance a lot

File: chapter_10_codes/sensor_sim_gazebo/urdf/imu.xacro (robot description, xacro)
@@ -38,5 +38,5 @@
       <plugin name="sensor" filename="libgazebo_ros_imu.so">
         <alwaysOn>true</alwaysOn>
-        <bodyName>${parent}</bodyName>
+        <bodyName>gps</bodyName>
         <topicName>imu</topicName>
         <serviceName>imu_service</serviceName>

File: chapter_10_codes/sensor_sim_gazebo/urdf/sensor.xacro (robot description, xacro)
@@ -3,5 +3,5 @@
   <xacro:property name="height1" value="0.2" />
   <xacro:property name="width" value="0.2" />
-  <xacro:property name="parent" value="base_footprint" />
+  <xacro:property name="parent" value="gps" />
  <!-- Used for fixing robot to Gazebo 'base_link' -->
   <!-- <link name="${parent}"/> -->

Commit message: Updating simulation_handler to use RTK topics

File: chapter_10_codes/sensor_sim_gazebo/urdf/imu.xacro (robot description, xacro)
@@ -13,5 +13,5 @@
         <material name="white">
           <color rgba="1 1 1 1" />
-        </material>
+        </material>ro
       </visual>
       <collision>

File: chapter_10_codes/sensor_sim_gazebo/urdf/sensor.xacro (robot description, xacro)
@@ -13,5 +13,5 @@
   <link name="sensor">
     <collision>
-      <origin xyz="0 0 ${height1/2}" rpy="0 0 0"/>
+      <origin xyz="-1 0 ${height1/2}" rpy="0 0 0"/>
       <geometry>
         <box size="${width} ${width} ${height1}"/>
@@ -19,5 +19,5 @@
     </collision>
     <visual>
-      <origin xyz="0 0 ${height1/2}" rpy="0 0 0"/>
+      <origin xyz="-1 0 ${height1/2}" rpy="0 0 0"/>
       <geometry>
         <box size="${width} ${width} ${height1}"/>
@@ -26,10 +26,10 @@
     </visual>
     <inertial>
-      <origin xyz="0 0 1" rpy="0 0 0"/>
-      <mass value="1"/>
+      <origin xyz="-1 0 1" rpy="0 0 0"/>
+      <mass value="0.000001"/>
       <inertia
-        ixx="1.0" ixy="0.0" ixz="0.0"
-        iyy="1.0" iyz="0.0"
-        izz="1.0"/>
+        ixx="0.000001" ixy="0.0" ixz="0.0"
+        iyy="0.000001" iyz="0.0"
+        izz="0.000001"/>
     </inertial>
   </link>
